File: PCB/fpga_bank4.kicad_sch (KiCad schematic)
At the start: 14 parts, among them U2 XC7A50T-FGG484

Commit message: Version 1.2 routed
Other:
- title: FPGA Bank 216 (MGT/PCIe) -> Pi 5 - Artix XC7A50T - PCIe FPGA Hat
Changed lines of the file:
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@@
 	(paper "A4")
 	(title_block
-		(title "FPGA Bank 216 (MGT/PCIe)")
-		(date "2024-03-24")
-		(rev "1.1")
+		(title "Pi 5 - Artix XC7A50T - PCIe FPGA Hat")
+		(date "2025-07-17")
+		(rev "1.2")
 		(company "George Smart, M1GEO")
 		(comment 1 "https://github.com/m1geo/Pi5-Artix-FPGA-Hat")
