File: PCB/fpga_top.kicad_sch (KiCad schematic)
At the start: 7 parts, among them X1 50MHz

Commit message: Version 1.2 routed
Other:
- title: FPGA Top Sheet -> Pi 5 - Artix XC7A50T - PCIe FPGA Hat
Changed lines of the file:
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@@
 	(paper "A4")
 	(title_block
-		(title "FPGA Top Sheet")
-		(date "2024-03-24")
-		(rev "1.1")
+		(title "Pi 5 - Artix XC7A50T - PCIe FPGA Hat")
+		(date "2025-07-17")
+		(rev "1.2")
 		(company "George Smart, M1GEO")
 		(comment 1 "https://github.com/m1geo/Pi5-Artix-FPGA-Hat")

Commit message: Updating LEDs footprint and Resistors value
Parts:
- D2: footprint LED_SMD:LED_0402_1005Metric -> LED_SMD:LED_0603_1608Metric
Changed lines of the file:
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@@
 			)
 		)
-		(property "Footprint" "LED_SMD:LED_0402_1005Metric"
+		(property "Footprint" "LED_SMD:LED_0603_1608Metric"
 			(at 194.945 54.61 0)
 			(effects
