File: PCB/fpga_bank2.kicad_sch (KiCad schematic)
At the start: 17 parts, among them J5 MIPI0, J6 MIPI1, U2 XC7A50T-FGG484

Commit message: connecting JTAG and other non diff pins, routing
Connections:
- net +3V3: no longer C38.2, C47.2, C48.2, C49.2, C50.2, C53.2, C58.2, C59.2, C66.2, C67.2
- net BANK_15_VCC: now also C38.2, C47.2, C48.2, C49.2, C50.2, J5.22 (Pin_22), J6.22 (Pin_22)
- net BANK_16_VCC: now also C53.2, C58.2, C59.2, C66.2, C67.2
- net GND: now also J5.1 (Pin_1), J5.10 (Pin_10), J5.13 (Pin_13), J5.16 (Pin_16), J5.19 (Pin_19), J5.4 (Pin_4), J5.7 (Pin_7), J6.1 (Pin_1), J6.10 (Pin_10), J6.13 (Pin_13), J6.16 (Pin_16), J6.19 (Pin_19), J6.4 (Pin_4), J6.7 (Pin_7)
- net SCL0: now reaches U2.B21 (IO_L21P_T3_DQS_16)
- net SCL0: now also J5.20 (Pin_20), J6.20 (Pin_20)
- net MIPI1_CAM_GPIO1: now reaches U2.B22 (IO_L20N_T3_16)
- net MIPI1_CAM_GPIO1: now also J6.18 (Pin_18)
- net SDA0: now reaches U2.C20 (IO_L19N_T3_VREF_16)
- net SDA0: now also J5.21 (Pin_21), J6.21 (Pin_21)
- net MIPI1_CAM_GPIO0: now reaches U2.D20 (IO_L19P_T3_16)
- net MIPI1_CAM_GPIO0: now also J6.17 (Pin_17)
- net MIPI0_CAM_GPIO0: now reaches U2.F19 (IO_L18P_T2_16)
- net MIPI0_CAM_GPIO0: now also J5.17 (Pin_17)
- net MIPI0_CAM_GPIO1: now reaches U2.F20 (IO_L18N_T2_16)
- net MIPI0_CAM_GPIO1: now also J5.18 (Pin_18)
- no-connect marks 56 -> 50
Other:
- moved on the sheet: J5, J6

Commit message: Version 1.2 routed
Other:
- title: FPGA Banks 15 & 16 -> Pi 5 - Artix XC7A50T - PCIe FPGA Hat
Changed lines of the file:
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@@
 	(paper "A4")
 	(title_block
-		(title "FPGA Banks 15 & 16")
-		(date "2024-03-24")
-		(rev "1.1")
+		(title "Pi 5 - Artix XC7A50T - PCIe FPGA Hat")
+		(date "2025-07-17")
+		(rev "1.2")
 		(company "George Smart, M1GEO")
 		(comment 1 "https://github.com/m1geo/Pi5-Artix-FPGA-Hat")

Commit message: MIPI conectors should be now compatible with C597981
Connections:
- net BANK_15_VCC: now also J5.1 (Pin_1), J6.1 (Pin_1); no longer J5.22 (Pin_22), J6.22 (Pin_22)
- net GND: now also J5.22 (Pin_22), J6.22 (Pin_22); no longer J5.1 (Pin_1), J6.1 (Pin_1)
- net MIPI0_CAM_GPIO0: now also J5.6 (Pin_6), U2.B21 (IO_L21P_T3_DQS_16); no longer J5.17 (Pin_17), U2.F19 (IO_L18P_T2_16)
- net MIPI0_CAM_GPIO1: now also J5.5 (Pin_5), U2.C20 (IO_L19N_T3_VREF_16); no longer J5.18 (Pin_18), U2.F20 (IO_L18N_T2_16)
- net MIPI0_CK+: now also J5.15 (Pin_15); no longer J5.8 (Pin_8)
- net MIPI0_CK-: now also J5.14 (Pin_14); no longer J5.9 (Pin_9)
- net MIPI0_D0+: now also J5.21 (Pin_21), U2.L19 (IO_L14P_T2_SRCC_15); no longer J5.2 (Pin_2), U2.N18 (IO_L17P_T2_A26_15)
- net MIPI0_D0-: now also J5.20 (Pin_20), U2.L20 (IO_L14N_T2_SRCC_15); no longer J5.3 (Pin_3), U2.N19 (IO_L17N_T2_A25_15)
- net MIPI0_D1+: now also J5.9 (Pin_9), U2.N18 (IO_L17P_T2_A26_15); no longer J5.14 (Pin_14), U2.L19 (IO_L14P_T2_SRCC_15)
- net MIPI0_D1-: now also J5.8 (Pin_8), U2.N19 (IO_L17N_T2_A25_15); no longer J5.15 (Pin_15), U2.L20 (IO_L14N_T2_SRCC_15)
- net MIPI0_D2+: now also J5.12 (Pin_12), U2.M18 (IO_L16P_T2_A28_15); no longer J5.11 (Pin_11), U2.N22 (IO_L15P_T2_DQS_15)
- net MIPI0_D2-: now also J5.11 (Pin_11), U2.L18 (IO_L16N_T2_A27_15); no longer J5.12 (Pin_12), U2.M22 (IO_L15N_T2_DQS_ADV_B_15)
- net MIPI0_D3+: now also J5.18 (Pin_18), U2.N22 (IO_L15P_T2_DQS_15); no longer J5.5 (Pin_5), U2.M18 (IO_L16P_T2_A28_15)
- net MIPI0_D3-: now also J5.17 (Pin_17), U2.M22 (IO_L15N_T2_DQS_ADV_B_15); no longer J5.6 (Pin_6), U2.L18 (IO_L16N_T2_A27_15)
- net MIPI1_CAM_GPIO0: now also J6.6 (Pin_6); no longer J6.17 (Pin_17)
- net MIPI1_CAM_GPIO1: now also J6.5 (Pin_5); no longer J6.18 (Pin_18)
- net MIPI1_CK+: now also J6.15 (Pin_15); no longer J6.8 (Pin_8)
- net MIPI1_CK-: now also J6.14 (Pin_14); no longer J6.9 (Pin_9)
- net MIPI1_D0+: now also J6.21 (Pin_21), U2.H20 (IO_L8P_T1_AD10P_15); no longer J6.2 (Pin_2), U2.M21 (IO_L10P_T1_AD11P_15)
- net MIPI1_D0-: now also J6.20 (Pin_20), U2.G20 (IO_L8N_T1_AD10N_15); no longer J6.3 (Pin_3), U2.L21 (IO_L10N_T1_AD11N_15)
- net MIPI1_D1+: now also J6.9 (Pin_9), U2.M21 (IO_L10P_T1_AD11P_15); no longer J6.14 (Pin_14), U2.H20 (IO_L8P_T1_AD10P_15)
- net MIPI1_D1-: now also J6.8 (Pin_8), U2.L21 (IO_L10N_T1_AD11N_15); no longer J6.15 (Pin_15), U2.G20 (IO_L8N_T1_AD10N_15)
- net MIPI1_D2+: now also J6.12 (Pin_12), U2.K21 (IO_L9P_T1_DQS_AD3P_15); no longer J6.11 (Pin_11), U2.J22 (IO_L7P_T1_AD2P_15)
- net MIPI1_D2-: now also J6.11 (Pin_11), U2.K22 (IO_L9N_T1_DQS_AD3N_15); no longer J6.12 (Pin_12), U2.H22 (IO_L7N_T1_AD2N_15)
- net MIPI1_D3+: now also J6.18 (Pin_18), U2.J22 (IO_L7P_T1_AD2P_15); no longer J6.5 (Pin_5), U2.K21 (IO_L9P_T1_DQS_AD3P_15)
- net MIPI1_D3-: now also J6.17 (Pin_17), U2.H22 (IO_L7N_T1_AD2N_15); no longer J6.6 (Pin_6), U2.K22 (IO_L9N_T1_DQS_AD3N_15)
- net SCL0: now also J5.3 (Pin_3), J6.3 (Pin_3), U2.F20 (IO_L18N_T2_16); no longer J5.20 (Pin_20), J6.20 (Pin_20), U2.B21 (IO_L21P_T3_DQS_16)
- net SDA0: now also J5.2 (Pin_2), J6.2 (Pin_2), U2.F19 (IO_L18P_T2_16); no longer J5.21 (Pin_21), J6.21 (Pin_21), U2.C20 (IO_L19N_T3_VREF_16)
Other:
- moved on the sheet: J5, J6

Commit message: Updating LEDs footprint and Resistors value
Parts:
- J5: value MIPI0 -> C597981; LCSC (none) -> C597981
- J6: value MIPI1 -> C597981; LCSC (none) -> C597981
Changed lines of the file:
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@@
 			)
 		)
-		(property "Value" "MIPI0"
+		(property "Value" "C597981"
 			(at 203.2 128.2699 0)
 			(effects
@@
 			)
 		)
-		(property "Datasheet" "~"
+		(property "Datasheet" "https://lcsc.com/datasheet/lcsc_datasheet_2410121851_HRS-FH12-22S-0-5SH-55_C597981.pdf"
 			(at 204.47 128.27 0)
 			(effects
@@
 		)
 		(property "Description" "Generic connector, single row, 01x22, script generated"
+			(at 204.47 128.27 0)
+			(effects
+				(font
+					(size 1.27 1.27)
+				)
+				(hide yes)
+			)
+		)
+		(property "LCSC" "C597981"
 			(at 204.47 128.27 0)
 			(effects
@@
 			)
 		)
-		(property "Value" "MIPI1"
+		(property "Value" "C597981"
 			(at 242.57 128.2699 0)
 			(effects
@@
 			)
 		)
-		(property "Datasheet" "~"
+		(property "Datasheet" "https://lcsc.com/datasheet/lcsc_datasheet_2410121851_HRS-FH12-22S-0-5SH-55_C597981.pdf"
 			(at 243.84 128.27 0)
 			(effects
@@
 			(at 243.84 128.27 0)
 			(effects
+				(font
+					(size 1.27 1.27)
+				)
+				(hide yes)
+			)
+		)
+		(property "LCSC" "C597981"
+			(at 243.84 128.27 0)
+			(effects

Commit message: updating connector
Parts:
- J5, J6: footprint Connector_FFC-FPC:Amphenol_F32Q-1A7x1-11022_1x22-1MP_P0.5mm_Horizontal -> FHT12:CONN_FH12-22S-0.5SH55_HIR
Changed lines of the file:
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@@
 			)
 		)
-		(property "Footprint" "Connector_FFC-FPC:Amphenol_F32Q-1A7x1-11022_1x22-1MP_P0.5mm_Horizontal"
+		(property "Footprint" "FHT12:CONN_FH12-22S-0.5SH55_HIR"
 			(at 204.47 128.27 0)
 			(effects
@@
 			)
 		)
-		(property "Footprint" "Connector_FFC-FPC:Amphenol_F32Q-1A7x1-11022_1x22-1MP_P0.5mm_Horizontal"
+		(property "Footprint" "FHT12:CONN_FH12-22S-0.5SH55_HIR"
 			(at 243.84 128.27 0)
 			(effects
